File: VideoTimingBoard.sch (KiCad schematic (older format))
At the start: 37 parts, among them U1 MC44144, U2 LM1881, U3 SN74LVC3G04, U4 TLV3502

Commit message: Design complete.
Parts:
- J1: footprint Connector_PinHeader_1.27mm:PinHeader_1x15_P1.27mm_Vertical -> Connector_PinHeader_1.27mm:PinHeader_1x17_P1.27mm_Vertical
- R10: value 10K -> 150R
- U3: value SN74LVC3G04 -> SN74LVC1GU04
- U4: footprint Package_TO_SOT_SMD:SOT-23-8_Handsoldering -> Package_SO:SOIC-8_3.9x4.9mm_P1.27mm
Connections:
- net labels added: 4FSC-BIAS, FSC-BIAS
Changed lines of the file:
@@
 F 0 "U4" H 6050 5100 60  0000 L CNN
 F 1 "TLV3502" H 5900 4950 60  0000 L CNN
-F 2 "Package_TO_SOT_SMD:SOT-23-8_Handsoldering" H 5800 4750 50  0001 C CNN
+F 2 "Package_SO:SOIC-8_3.9x4.9mm_P1.27mm" H 5800 4750 50  0001 C CNN
 F 3 "http://www.ti.com/lit/ds/symlink/tlv3501.pdf" H 5800 4750 50  0001 C CNN
 	1    5800 4750
@@
 L Device:C_Small C8
 U 1 1 5C99D691
-P 2650 5450
+P 2950 5450
 AR Path="/5C99D691" Ref="C8"  Part="1"
 AR Path="/5CAADBB8/5C99D691" Ref="C?"  Part="1"
-F 0 "C8" V 2400 5450 50  0000 C CNN
-F 1 "1nF" V 2500 5450 50  0000 C CNN
-F 2 "Capacitor_SMD:C_0402_1005Metric" H 2650 5450 50  0001 C CNN
-F 3 "~" H 2650 5450 50  0001 C CNN
-	1    2650 5450
+F 0 "C8" V 2700 5450 50  0000 C CNN
+F 1 "1nF" V 2800 5450 50  0000 C CNN
+F 2 "Capacitor_SMD:C_0402_1005Metric" H 2950 5450 50  0001 C CNN
+F 3 "~" H 2950 5450 50  0001 C CNN
+	1    2950 5450
 	0    1    1    0
 $EndComp
-Text Label 3050 5450 0    50   ~ 0
-FSC
+Text Label 3200 5450 0    50   ~ 0
+FSC-BIAS
 $Comp
 L power:GND #PWR05
@@
 	1    0    0    -1
 $EndComp
-Wire Wire Line
-	2550 5450 2450 5450
 $Comp
 L Device:R_Small R5
@@
 AR Path="/5CAADBB8/5C99D723" Ref="U?"  Part="1"
 F 0 "U3" H 6050 2300 50  0000 L CNN
-F 1 "SN74LVC3G04" H 6050 2200 50  0000 L CNN
+F 1 "SN74LVC1GU04" H 6050 2200 50  0000 L CNN
 F 2 "Package_SO:Texas_R-PDSO-N5" H 6000 1950 50  0001 C CNN
 F 3 "http://www.ti.com/lit/ds/symlink/sn74ahc1g04.pdf" H 6000 1950 50  0001 C CNN
@@
 F 0 "U4" H 6150 6550 60  0000 C CNN
 F 1 "TLV3502" H 6150 6400 60  0000 C CNN
-F 2 "Package_TO_SOT_SMD:SOT-23-8_Handsoldering" H 5700 5100 50  0001 C CNN
+F 2 "Package_SO:SOIC-8_3.9x4.9mm_P1.27mm" H 5700 5100 50  0001 C CNN
 F 3 "http://www.ti.com/lit/ds/symlink/tlv3501.pdf" H 5650 5250 50  0001 C CNN
 	2    5800 6200
@@
 L Device:C_Small C9
 U 1 1 5C99D7F3
-P 2650 5700
+P 2950 5700
 AR Path="/5C99D7F3" Ref="C9"  Part="1"
 AR Path="/5CAADBB8/5C99D7F3" Ref="C?"  Part="1"
-F 0 "C9" V 2800 5700 50  0000 C CNN
-F 1 "1nF" V 2900 5700 50  0000 C CNN
-F 2 "Capacitor_SMD:C_0402_1005Metric" H 2650 5700 50  0001 C CNN
-F 3 "~" H 2650 5700 50  0001 C CNN
-	1    2650 5700
+F 0 "C9" V 3100 5700 50  0000 C CNN
+F 1 "1nF" V 3200 5700 50  0000 C CNN
+F 2 "Capacitor_SMD:C_0402_1005Metric" H 2950 5700 50  0001 C CNN
+F 3 "~" H 2950 5700 50  0001 C CNN
+	1    2950 5700
 	0    1    1    0
 $EndComp
@@
 	3650 6350 3650 5700
 Wire Wire Line
-	3650 5700 2750 5700
-Wire Wire Line
 	3650 6350 4400 6350
 Wire Wire Line
-	2550 5700 2450 5700
-Wire Wire Line
 	3650 5450 3650 5100
 Wire Wire Line
-	2750 5450 3650 5450
-Wire Wire Line
 	3650 5100 4400 5100
-Text Label 3050 5700 0    50   ~ 0
-4FSC
+Text Label 3200 5700 0    50   ~ 0
+4FSC-BIAS
 Connection ~ 4400 5100
 Wire Wire Line
@@
 AR Path="/5C99D856" Ref="R10"  Part="1"
 F 0 "R10" H 8509 1746 50  0000 L CNN
-F 1 "10K" H 8509 1655 50  0000 L CNN
+F 1 "150R" H 8509 1655 50  0000 L CNN
 F 2 "Resistor_SMD:R_0603_1608Metric_Pad1.05x0.95mm_HandSolder" H 8450 1700 50  0001 C CNN
 F 3 "~" H 8450 1700 50  0001 C CNN
@@
 F 0 "J1" H 10650 2900 50  0000 C CNN
 F 1 "~" H 10700 2476 50  0000 C CNN
-F 2 "Connector_PinHeader_1.27mm:PinHeader_1x15_P1.27mm_Vertical" H 10650 1950 50  0001 C CNN
+F 2 "Connector_PinHeader_1.27mm:PinHeader_1x17_P1.27mm_Vertical" H 10650 1950 50  0001 C CNN
 F 3 "~" H 10650 1950 50  0001 C CNN
 	1    10650 1950
@@
 Text Label 9600 1350 0    50   ~ 0
 CVBS-CLAMPED
+Wire Wire Line
+	3650 5450 3050 5450
+Wire Wire Line
+	2450 5450 2850 5450
+Wire Wire Line
+	2450 5700 2850 5700
+Wire Wire Line
+	3050 5700 3650 5700
+Text Label 2600 5450 0    50   ~ 0
+FSC
+Text Label 2600 5700 0    50   ~ 0
+4FSC
 $EndSCHEMATC

Commit message: Changed .05" pinheaders to .1" Removed CVBS clamp The MC44144 and LM1881 are separately AC-coupled to the CVBS signal.
Parts:
- removed D1: BAT54, Package_TO_SOT_SMD:SOT-23, symbol Schottky:D_Schottky
- added C18: 0.1uF, Capacitor_SMD:C_0402_1005Metric, symbol Device:C_Small
- J1: footprint Connector_PinHeader_1.27mm:PinHeader_1x17_P1.27mm_Vertical -> Connector_PinHeader_2.54mm:PinHeader_1x17_P2.54mm_Vertical
- R1: value 75R -> 0R
Connections:
- net labels added: CVBS, FSC1
- net labels removed: CVBS-CLAMPED, CVBS-IN
- wire segments 156 -> 152
Changed lines of the file:
@@
 L Device:C_Small C3
 U 1 1 5C99D62F
-P 1650 1400
+P 2250 1550
 AR Path="/5C99D62F" Ref="C3"  Part="1"
 AR Path="/5CAADBB8/5C99D62F" Ref="C?"  Part="1"
-F 0 "C3" V 1902 1400 50  0000 C CNN
-F 1 "0.1uF" V 1811 1400 50  0000 C CNN
-F 2 "Capacitor_SMD:C_0402_1005Metric" H 1688 1250 50  0001 C CNN
-F 3 "~" H 1650 1400 50  0001 C CNN
-	1    1650 1400
-	0    -1   -1   0
+F 0 "C3" V 2502 1550 50  0000 C CNN
+F 1 "0.1uF" V 2411 1550 50  0000 C CNN
+F 2 "Capacitor_SMD:C_0402_1005Metric" H 2288 1400 50  0001 C CNN
+F 3 "~" H 2250 1550 50  0001 C CNN
+	1    2250 1550
+	-1   0    0    1
 $EndComp
 $Comp
@@
 Wire Wire Line
 	2050 4850 2050 5100
-Text Label 550  5450 0    50   ~ 0
-CVBS-CLAMPED
 $Comp
 L Device:C_Small C8
@@
 	1    0    0    -1
 $EndComp
-Wire Wire Line
-	2250 1400 2250 1750
 $Comp
 L Device:R_Small R4
@@
 	1850 2200 1850 2300
 $Comp
-L Device:R_Small R1
-U 1 1 5C99D751
-P 1300 1650
-AR Path="/5C99D751" Ref="R1"  Part="1"
-AR Path="/5CAADBB8/5C99D751" Ref="R?"  Part="1"
-F 0 "R1" V 1104 1650 50  0000 C CNN
-F 1 "75R" V 1195 1650 50  0000 C CNN
-F 2 "Resistor_SMD:R_0603_1608Metric_Pad1.05x0.95mm_HandSolder" H 1300 1650 50  0001 C CNN
-F 3 "~" H 1300 1650 50  0001 C CNN
-	1    1300 1650
-	-1   0    0    1
-$EndComp
-Wire Wire Line
-	1300 1550 1300 1400
-Connection ~ 1300 1400
-$Comp
-L power:GND #PWR03
-U 1 1 5C99D75A
-P 1300 1800
-AR Path="/5C99D75A" Ref="#PWR03"  Part="1"
-AR Path="/5CAADBB8/5C99D75A" Ref="#PWR?"  Part="1"
-F 0 "#PWR03" H 1300 1550 50  0001 C CNN
-F 1 "GND" H 1305 1627 50  0000 C CNN
-F 2 "" H 1300 1800 50  0001 C CNN
-F 3 "" H 1300 1800 50  0001 C CNN
-	1    1300 1800
-	1    0    0    -1
-$EndComp
-Wire Wire Line
-	1300 1800 1300 1750
-$Comp
 L Device:C_Small C14
 U 1 1 5C99D761
@@
 Wire Wire Line
 	1650 4500 1650 4700
-Wire Wire Line
-	1300 1400 1550 1400
 $Comp
 L Device:C_Small C10
@@
 Text Notes 2350 4750 0    50   ~ 0
 14.31818 MHz (NTSC)\n17.734475 MHz (PAL)
-$Comp
-L Schottky:D_Schottky D?
-U 1 1 5C99D7B3
-P 1900 1650
-AR Path="/5CAADBB8/5C99D7B3" Ref="D?"  Part="1"
-AR Path="/5C99D7B3" Ref="D1"  Part="1"
-F 0 "D1" V 1854 1729 50  0000 L CNN
-F 1 "BAT54" V 1945 1729 50  0000 L CNN
-F 2 "Package_TO_SOT_SMD:SOT-23" H 1900 1650 50  0001 C CNN
-F 3 "~" H 1900 1650 50  0001 C CNN
-	1    1900 1650
-	0    1    1    0
-$EndComp
-$Comp
-L power:GND #PWR06
-U 1 1 5C99D7BA
-P 1900 1800
-AR Path="/5C99D7BA" Ref="#PWR06"  Part="1"
-AR Path="/5CAADBB8/5C99D7BA" Ref="#PWR?"  Part="1"
-F 0 "#PWR06" H 1900 1550 50  0001 C CNN
-F 1 "GND" H 1905 1627 50  0000 C CNN
-F 2 "" H 1900 1800 50  0001 C CNN
-F 3 "" H 1900 1800 50  0001 C CNN
-	1    1900 1800
-	1    0    0    -1
-$EndComp
-Wire Wire Line
-	1750 1400 1900 1400
-Wire Wire Line
-	1900 1500 1900 1400
-Connection ~ 1900 1400
-Wire Wire Line
-	1900 1400 2250 1400
-Wire Wire Line
-	2250 950  2250 1400
-Connection ~ 2250 1400
 Text Label 2050 5050 1    50   ~ 0
 XTAL
@@
 F 0 "J1" H 10650 2900 50  0000 C CNN
 F 1 "~" H 10700 2476 50  0000 C CNN
-F 2 "Connector_PinHeader_1.27mm:PinHeader_1x17_P1.27mm_Vertical" H 10650 1950 50  0001 C CNN
+F 2 "Connector_PinHeader_2.54mm:PinHeader_1x17_P2.54mm_Vertical" H 10650 1950 50  0001 C CNN
 F 3 "~" H 10650 1950 50  0001 C CNN
 	1    10650 1950
@@
 Text Label 3800 1950 2    50   ~ 0
 FIELD
-Wire Wire Line
-	800  950  2250 950
-Wire Wire Line
-	800  1400 1300 1400
-Text Label 800  1400 0    50   ~ 0
-CVBS-IN
-Text Label 800  950  0    50   ~ 0
-CVBS-CLAMPED
-Wire Wire Line
-	550  5450 1200 5450
+Text Label 1200 1200 0    50   ~ 0
+CVBS
 Wire Wire Line
 	550  5700 1200 5700
 Text Label 10000 3850 0    50   ~ 0
-CVBS-IN
+CVBS
 Text Label 9600 2450 0    50   ~ 0
 GND
 Text Label 9600 2350 0    50   ~ 0
-FSC
+FSC1
 Wire Wire Line
 	10450 1250 9600 1250
@@
 GND
 Text Label 9600 1350 0    50   ~ 0
-CVBS-CLAMPED
+CVBS
 Wire Wire Line
 	3650 5450 3050 5450
@@
 Text Label 2600 5700 0    50   ~ 0
 4FSC
+Wire Wire Line
+	2250 1650 2250 1750
+Wire Wire Line
+	1200 1200 2250 1200
+Wire Wire Line
+	2250 1200 2250 1450
+$Comp
+L Device:C_Small C18
+U 1 1 5D6B0B47
+P 950 5450
+AR Path="/5D6B0B47" Ref="C18"  Part="1"
+AR Path="/5CAADBB8/5D6B0B47" Ref="C?"  Part="1"
+F 0 "C18" V 1202 5450 50  0000 C CNN
+F 1 "0.1uF" V 1111 5450 50  0000 C CNN
+F 2 "Capacitor_SMD:C_0402_1005Metric" H 988 5300 50  0001 C CNN
+F 3 "~" H 950 5450 50  0001 C CNN
+	1    950  5450
+	0    -1   -1   0
+$EndComp
+Wire Wire Line
+	1050 5450 1200 5450
+Wire Wire Line
+	850  5450 550  5450
+Text Label 550  5450 0    50   ~ 0
+CVBS
+$Comp
+L Device:R_Small R1
+U 1 1 5D6BC863
+P 7800 3250
+AR Path="/5D6BC863" Ref="R1"  Part="1"
+AR Path="/5CAADBB8/5D6BC863" Ref="R?"  Part="1"
+F 0 "R1" V 7700 3250 50  0000 C CNN
+F 1 "0R" V 7600 3250 50  0000 C CNN
+F 2 "Resistor_SMD:R_0603_1608Metric_Pad1.05x0.95mm_HandSolder" H 7800 3250 50  0001 C CNN
+F 3 "~" H 7800 3250 50  0001 C CNN
+	1    7800 3250
+	0    -1   -1   0
+$EndComp
+Text Label 7550 3250 0    50   ~ 0
+FSC
+Text Label 8100 3250 2    50   ~ 0
+FSC1
+Wire Wire Line
+	7550 3250 7700 3250
+Wire Wire Line
+	7900 3250 8100 3250
 $EndSCHEMATC

Commit message: Changed jumpers
Parts:
- added R11: 0R, Resistor_SMD:R_0603_1608Metric_Pad1.05x0.95mm_HandSolder, symbol Device:R_Small
- added R12: R0, Resistor_SMD:R_0603_1608Metric_Pad1.05x0.95mm_HandSolder, symbol Device:R_Small
- U3: footprint Package_SO:Texas_R-PDSO-N5 -> Package_TO_SOT_SMD:SOT-23-5_HandSoldering
Connections:
- wire segments 152 -> 156
Other:
- note added: "Jumpers"
Changed lines of the file:
@@
 F 0 "U3" H 6050 2300 50  0000 L CNN
 F 1 "SN74LVC1GU04" H 6050 2200 50  0000 L CNN
-F 2 "Package_SO:Texas_R-PDSO-N5" H 6000 1950 50  0001 C CNN
+F 2 "Package_TO_SOT_SMD:SOT-23-5_HandSoldering" H 6000 1950 50  0001 C CNN
 F 3 "http://www.ti.com/lit/ds/symlink/sn74ahc1g04.pdf" H 6000 1950 50  0001 C CNN
 	1    5900 1950
@@
 L Device:R_Small R1
 U 1 1 5D6BC863
-P 7800 3250
+P 7750 3300
 AR Path="/5D6BC863" Ref="R1"  Part="1"
 AR Path="/5CAADBB8/5D6BC863" Ref="R?"  Part="1"
-F 0 "R1" V 7700 3250 50  0000 C CNN
-F 1 "0R" V 7600 3250 50  0000 C CNN
-F 2 "Resistor_SMD:R_0603_1608Metric_Pad1.05x0.95mm_HandSolder" H 7800 3250 50  0001 C CNN
-F 3 "~" H 7800 3250 50  0001 C CNN
-	1    7800 3250
+F 0 "R1" V 7950 3300 50  0000 C CNN
+F 1 "0R" V 7850 3300 50  0000 C CNN
+F 2 "Resistor_SMD:R_0603_1608Metric_Pad1.05x0.95mm_HandSolder" H 7750 3300 50  0001 C CNN
+F 3 "~" H 7750 3300 50  0001 C CNN
+	1    7750 3300
 	0    -1   -1   0
 $EndComp
-Text Label 7550 3250 0    50   ~ 0
+Text Label 7300 3300 0    50   ~ 0
 FSC
-Text Label 8100 3250 2    50   ~ 0
+Text Label 8150 3300 2    50   ~ 0
 FSC1
-Wire Wire Line
-	7550 3250 7700 3250
-Wire Wire Line
-	7900 3250 8100 3250
+$Comp
+L Device:R_Small R11
+U 1 1 5D6D97DA
+P 7750 3600
+F 0 "R11" V 7554 3600 50  0000 C CNN
+F 1 "0R" V 7645 3600 50  0000 C CNN
+F 2 "Resistor_SMD:R_0603_1608Metric_Pad1.05x0.95mm_HandSolder" H 7750 3600 50  0001 C CNN
+F 3 "~" H 7750 3600 50  0001 C CNN
+	1    7750 3600
+	0    1    1    0
+$EndComp
+$Comp
+L Device:R_Small R12
+U 1 1 5D6D9880
+P 7750 3900
+F 0 "R12" V 7554 3900 50  0000 C CNN
+F 1 "R0" V 7645 3900 50  0000 C CNN
+F 2 "Resistor_SMD:R_0603_1608Metric_Pad1.05x0.95mm_HandSolder" H 7750 3900 50  0001 C CNN
+F 3 "~" H 7750 3900 50  0001 C CNN
+	1    7750 3900
+	0    1    1    0
+$EndComp
+Text Label 7300 3600 0    50   ~ 0
+VDD
+Text Label 8150 3600 2    50   ~ 0
+VDD
+Wire Wire Line
+	7300 3600 7650 3600
+Wire Wire Line
+	7850 3600 8150 3600
+Wire Wire Line
+	7300 3300 7650 3300
+Wire Wire Line
+	7850 3300 8150 3300
+Text Label 7300 3900 0    50   ~ 0
+VDD
+Text Label 8150 3900 2    50   ~ 0
+VDD
+Wire Wire Line
+	7300 3900 7650 3900
+Wire Wire Line
+	7850 3900 8150 3900
+Text Notes 7600 4100 0    50   ~ 0
+Jumpers
 $EndSCHEMATC
